Commit message: manual editted version

File: kuka_kr300_support/urdf/kr300r2500pro.urdf (robot description, URDF)
Before this commit: robot kuka_kr300r2500pro, 0 links, 0 joints
Links:
- added link base
- added link base_link, mass 2; collision mesh filename=package://kuka_kr300_support/meshes/kr300r2500pro/collision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; visual mesh filename=package://kuka_kr300_support/meshes/kr300r2500pro/visual/ba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
- added link link_1, mass 2; collision mesh filename=package://kuka_kr300_support/meshes/kr300r2500pro/collision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; visual mesh filename=package://kuka_kr300_support/meshes/kr300r2500pro/visual/li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
- added link link_2, mass 2; collision mesh filename=package://kuka_kr300_support/meshes/kr300r2500pro/collision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; visual mesh filename=package://kuka_kr300_support/meshes/kr300r2500pro/visual/li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
- added link link_3, mass 2; collision mesh filename=package://kuka_kr300_support/meshes/kr300r2500pro/collision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; visual mesh filename=package://kuka_kr300_support/meshes/kr300r2500pro/visual/li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
- added link link_4, mass 2; collision mesh filename=package://kuka_kr300_support/meshes/kr300r2500pro/collision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; visual mesh filename=package://kuka_kr300_support/meshes/kr300r2500pro/visual/li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
- added link link_5, mass 2; collision mesh filename=package://kuka_kr300_support/meshes/kr300r2500pro/collision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; visual mesh filename=package://kuka_kr300_support/meshes/kr300r2500pro/visual/li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
- added link link_6, mass 2; collision mesh filename=package://kuka_kr300_support/meshes/kr300r2500pro/collision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; visual mesh filename=package://kuka_kr300_support/meshes/kr300r2500pro/visual/li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
- added link tool0
Joints:
- added joint base_link-base: type fixed, parent base_link, child base, origin xyz=0 0 0 rpy=0 0 0
- added joint joint_a1: type revolute, parent base_link, child link_1, origin xyz=0 0 0.675 rpy=0 0 0, axis 0 0 -1, limit lower=-3.22885911619 upper=3.22885911619 effort=0 velocity=2.72271363311
- added joint joint_a2: type revolute, parent link_1, child link_2, origin xyz=0.35 0 0 rpy=0 0 0, axis 0 1 0, limit lower=-2.70526034059 upper=0.610865238198 effort=0 velocity=2.72271363311
- added joint joint_a3: type revolute, parent link_2, child link_3, origin xyz=1.150 0 0 rpy=0 0 0, axis 0 1 0, limit lower=-2.26892802759 upper=2.68780704807 effort=0 velocity=2.72271363311
- added joint joint_a4: type revolute, parent link_3, child link_4, origin xyz=1.0 0 -0.041 rpy=0 0 0, axis -1 0 0, limit lower=-6.10865238198 upper=6.10865238198 effort=0 velocity=5.75958653158
- added joint joint_a5: type revolute, parent link_4, child link_5, origin xyz=0 0 0 rpy=0 0 0, axis 0 1 0, limit lower=-2.26892802759 upper=2.26892802759 effort=0 velocity=5.75958653158
- added joint joint_a6: type revolute, parent link_5, child link_6, origin xyz=0 0 0 rpy=0 0 0, axis -1 0 0, limit lower=-6.10865238198 upper=6.10865238198 effort=0 velocity=10.7337748998
- added joint joint_a6-tool0: type fixed, parent link_6, child tool0, origin xyz=0.240 0 0 rpy=0 1.57079632679 0
